Commit message: feat: Updatedworks with 50hz freq with microros

File: jolie_humble/src/jolie_description/urdf/nebula_4wd.urdf.xacro (robot description, xacro)
@@ -8,5 +8,5 @@
     <xacro:property name="PI" value="3.1415926535897931"/>
     <xacro:property name="wheel_mass" value="0.105" />
-    <xacro:property name="wheel_radius" value="0.068337795" />
+    <xacro:property name="wheel_radius" value="0.028" />
     <xacro:property name="wheel_thickness" value="0.01905" />
     <xacro:property name="motor_shaft_radius" value="0.002" />
@@ -14,5 +14,5 @@
     <xacro:property name="shaft_mass" value="0.001" />
     <!-- parameters for chassis -->
-    <xacro:property name="chassis_radius" value="0.3"/>
+    <xacro:property name="chassis_radius" value="0.115"/>
     <xacro:property name="chassis_thickness" value="0.01"/>
     <xacro:include filename="$(find jolie_description)/urdf/common/materials.xacro"/>

Commit message: feat: update urdf lidar and twist mux (lidar error)

File: jolie_humble/src/jolie_description/urdf/nebula_4wd.urdf.xacro (robot description, xacro)
@@ -1,4 +1,18 @@
 <?xml version="1.0"?>
 <robot xmlns:xacro="http://www.ros.org/wiki/xacro" name="nebula_4wd">
+    <!-- Define inertial_cylinder macro here -->
+    <xacro:macro name="inertial_cylinder" params="mass length radius *origin">
+        <inertial>
+            <xacro:insert_block name="origin"/>
+            <mass value="${mass}" />
+            <inertia
+                ixx="${(1/12) * mass * (3*radius*radius + length*length)}"
+                ixy="0.0"
+                ixz="0.0"
+                iyy="${(1/12) * mass * (3*radius*radius + length*length)}"
+                iyz="0.0"
+                izz="${(1/2) * mass * (radius*radius)}" />
+            </inertial>
+    </xacro:macro>
     <!-- Argument -->
     <xacro:arg name="is_ignition" default="true"/>
@@ -21,4 +35,5 @@
     <xacro:include filename="$(find jolie_description)/urdf/common/omnidrive_base.urdf.xacro"/>
     <xacro:include filename="$(find jolie_description)/urdf/nebula_4wd_ros2_control.xacro"/>
+    <xacro:include filename="$(find jolie_description)/urdf/sensors/2d_lidar.xacro"/>
     <link name="base_link"></link>
     <joint name="base_to_chassis_joint" type="fixed">

File: jolie_humble/src/jolie_description/urdf/nebula_4wd_ros2_control.xacro (robot description, xacro)
@@ -89,4 +89,7 @@
             <parameters>$(find sirius_controller)/config/sirius_controllers.yaml</parameters>
         </plugin>
+        <plugin filename="ignition-gazebo-sensors-system" name="ignition::gazebo::systems::Sensors">
+            <render_engine>ogre2</render_engine>
+        </plugin>
         </xacro:if>
         <!-- ROS 2 Iron or above -->
@@ -95,4 +98,7 @@
             <parameters>$(find sirius_controller)/config/sirius_controllers.yaml</parameters>
         </plugin>
+        <plugin filename="gz-sim-sensors-system" name="gazebo::systems::Sensors">
+            <render_engine>ogre2</render_engine>
+        </plugin>
         </xacro:unless>
     </gazebo>

File: jolie_humble/src/jolie_description/urdf/sensors/2d_lidar.xacro (robot description, xacro)
@@ -7,10 +7,16 @@
 -->
 <robot xmlns:xacro="http://www.ros.org/wiki/xacro" >
+    <joint name="laser_joint" type="fixed">
+        <parent link="base_link"/>
+        <child link="laser_frame"/>
+        <origin xyz="-0.13 0 0.31" rpy="0 0 0"/>
+    </joint>
     <link name="laser_frame">
         <visual>
+            <origin xyz="0 0 0" rpy="0 0 0"/>
             <geometry>
                 <cylinder radius="0.05" length="0.04"/>
             </geometry>
-            <material name="red"/>
+            <material name="black"/>
         </visual>
         <collision>
@@ -24,29 +30,32 @@
     </link>
     <gazebo reference="laser_frame">
-        <material>Gazebo/Red</material>
-        <sensor name="laser" type="ray">
-            <pose> 0 0 0 0 0 0 </pose>
+        <material>Gazebo/Black</material>
+        <sensor name="laser" type="gpu_ray">
+            <always_on>true</always_on>
+            <pose>0 0 0 0 0 0</pose>
             <visualize>true</visualize>
-            <update_rate>10</update_rate>
+            <!-- Meningkatkan update rate agar lebih responsif -->
+            <update_rate>30</update_rate>
+            <gz_frame_id>laser_frame</gz_frame_id>
+            <topic>scan</topic>
             <ray>
                 <scan>
-                    <horizontal>
-                        <samples>360</samples>
-                        <min_angle>-3.14</min_angle>
-                        <max_angle>3.14</max_angle>
-                    </horizontal>
+                <horizontal>
+                    <samples>360</samples>
+                    <min_angle>-3.14</min_angle>
+                    <max_angle>3.14</max_angle>
+                </horizontal>
+                <!-- Tambahan parameter vertical -->
+                <vertical>
+                    <samples>1</samples>
+                    <min_angle>0</min_angle>
+                    <max_angle>0</max_angle>
+                </vertical>
                 </scan>
                 <range>
-                    <min>0.3</min>
-                    <max>12</max>
+                <min>0.3</min>
+                <max>12</max>
                 </range>
             </ray>
-            <plugin name="laser_controller" filename="libgazebo_ros_ray_sensor.so">
-                <ros>
-                    <argument>~/out:=scan</argument>
-                </ros>
-                <output_type>sensor_msgs/LaserScan</output_type>
-                <frame_name>laser_frame</frame_name>
-            </plugin>
         </sensor>
     </gazebo>

Commit message: feat: enhance launch files and add AMCL configuration for localization

File: jolie_humble/src/jolie_description/urdf/nebula_4wd.urdf.xacro (robot description, xacro)
@@ -42,4 +42,18 @@
         <child link="chassis_link"></child>
     </joint>
+    <link name="base_footprint">
+        <visual>
+            <origin xyz="0 0 0" rpy="0 0 0"/>
+            <geometry>
+                <sphere radius="0.01"/>
+            </geometry>
+            <material name="black"/>
+        </visual>
+    </link>
+    <joint name="base_footprint_to_base_link" type="fixed">
+        <origin xyz="0 0 0" rpy="0 0 0"/>
+        <parent link="base_footprint"/>
+        <child link="base_link"/>
+    </joint>
     <link name="chassis_link">
         <visual>

Commit message: feat: update URDF parameters and sensor configurations for improved accuracy

File: jolie_humble/src/jolie_description/urdf/nebula_4wd.urdf.xacro (robot description, xacro)
@@ -21,5 +21,5 @@
     <!-- parameters for wheel -->
     <xacro:property name="PI" value="3.1415926535897931"/>
-    <xacro:property name="wheel_mass" value="0.105" />
+    <xacro:property name="wheel_mass" value="0.0105" />
     <xacro:property name="wheel_radius" value="0.028" />
     <xacro:property name="wheel_thickness" value="0.01905" />

File: jolie_humble/src/jolie_description/urdf/sensors/2d_lidar.xacro (robot description, xacro)
@@ -10,5 +10,5 @@
         <parent link="base_link"/>
         <child link="laser_frame"/>
-        <origin xyz="-0.13 0 0.31" rpy="0 0 0"/>
+        <origin xyz="-0.13 0 0.15" rpy="0 0 0"/>
     </joint>
     <link name="laser_frame">
@@ -25,5 +25,5 @@
             </geometry>
         </collision>
-        <xacro:inertial_cylinder mass="0.1" length="0.04" radius="0.05">
+        <xacro:inertial_cylinder mass="0.01" length="0.04" radius="0.05">
             <origin xyz="0 0 0" rpy="0 0 0"/>
         </xacro:inertial_cylinder>
