Commit message: feat: update lidar pos.

File: jolie_humble/src/jolie_description/urdf/sensors/2d_lidar.xacro (robot description, xacro)
@@ -10,5 +10,5 @@
         <parent link="base_link"/>
         <child link="laser_frame"/>
-        <origin xyz="-0.13 0 0.15" rpy="0 0 0"/>
+        <origin xyz="0 0 0.15" rpy="0 0 0"/>
     </joint>
     <link name="laser_frame">
